File: _autosave-esp32c3-ev-board.kicad_sch (KiCad schematic)
At the start: 72 parts, among them IC1 SPX3819M5-L-3-3, IC2 ACS711EEXTK-31AB-T, IC3 ESP32-C3FH4, IC4 W25Q128JVSIQ, IC5 AH1390-HK4-7, J2 Battery Pos, J3 Barrel_Jack, J4 Conn_01x04_Pin, J5 USB_C_Receptacle_USB2.0, J6 Screw_Terminal_01x03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

Commit message: finishing touches
Parts:
- H7: footprint MountingHole:MountingHole_2.5mm_Pad -> MountingHole:MountingHole_2.2mm_M2
